File: software/BreadboardSimulator/data/circuit3.sch (KiCad schematic (older format))
At the start: 16 parts, among them Q1 Transistor, SW1 SwitchPush, U1-8 8pinChip

Commit message: add feature highlight selected pin
Connections:
- net +3V3: now also GND.1 (GND)
- net at CP1.2, D1.2 (A), SW1.1 (C): now also LED1.1 (K)
- removed net GND: GND.1 (GND), LED1.1 (K)
Other:
- moved on the sheet: D1, LED1
Changed lines of the file:
@@
 L SchemaBoard_Library:Diode D1
 U 1 1 5D3E50B4
-P 2550 5650
-F 0 "D1" H 2550 5866 50  0000 C CNN
-F 1 "Diode" H 2550 5775 50  0000 C CNN
-F 2 "" H 2550 5650 50  0001 C CNN
-F 3 "~" H 2550 5650 50  0001 C CNN
-	1    2550 5650
+P 2400 5650
+F 0 "D1" H 2400 5866 50  0000 C CNN
+F 1 "Diode" H 2400 5775 50  0000 C CNN
+F 2 "" H 2400 5650 50  0001 C CNN
+F 3 "~" H 2400 5650 50  0001 C CNN
+	1    2400 5650
 	1    0    0    -1
 $EndComp
@@
 L SchemaBoard_Library:GND GND
 U 1 1 5D3D0965
-P 950 6850
-F 0 "GND" H 950 6600 50  0001 C CNN
-F 1 "GND" H 955 6677 50  0000 C CNN
-F 2 "" H 950 6850 50  0001 C CNN
-F 3 "" H 950 6850 50  0001 C CNN
-	1    950  6850
+P 1550 4000
+F 0 "GND" H 1550 3750 50  0001 C CNN
+F 1 "GND" H 1555 3827 50  0000 C CNN
+F 2 "" H 1550 4000 50  0001 C CNN
+F 3 "" H 1550 4000 50  0001 C CNN
+	1    1550 4000
 	1    0    0    -1
 $EndComp
@@
 L SchemaBoard_Library:LED LED1
 U 1 1 5D3E5DAB
-P 1600 5650
-F 0 "LED1" H 1593 5866 50  0000 C CNN
-F 1 "LED" H 1593 5775 50  0000 C CNN
-F 2 "" H 1600 5650 50  0001 C CNN
-F 3 "~" H 1600 5650 50  0001 C CNN
-	1    1600 5650
+P 1350 6350
+F 0 "LED1" H 1343 6566 50  0000 C CNN
+F 1 "LED" H 1343 6475 50  0000 C CNN
+F 2 "" H 1350 6350 50  0001 C CNN
+F 3 "~" H 1350 6350 50  0001 C CNN
+	1    1350 6350
 	1    0    0    -1
 $EndComp
@@
 $EndComp
 Wire Wire Line
-	3050 1700 3050 3150
-Wire Wire Line
-	3050 3150 2500 3150
-Wire Wire Line
 	2100 2050 4150 2050
-Wire Wire Line
-	1800 2050 900  2050
 Wire Wire Line
 	900  2050 900  3300
@@
 	4200 5650 3950 5650
 Wire Wire Line
-	2700 5650 3150 5650
-Wire Wire Line
-	1750 5650 2400 5650
-Wire Wire Line
 	5650 6150 7350 6150
 Connection ~ 7350 6150
@@
 Wire Wire Line
 	3150 6850 3150 5650
-Connection ~ 3150 5650
 Wire Wire Line
 	3150 5650 3550 5650
-Wire Wire Line
-	1450 5650 950  5650
-Wire Wire Line
-	950  5650 950  6850
 Wire Wire Line
 	7100 3900 7850 3900
@@
 	4450 2050 5650 2050
 Wire Wire Line
-	2500 3300 2500 3150
+	1200 6350 900  6350
+Connection ~ 3150 5650
 Wire Wire Line
-	900  3300 2500 3300
+	2550 5650 3150 5650
+Wire Wire Line
+	2250 5650 1850 5650
+Wire Wire Line
+	1850 5650 1850 6350
+Wire Wire Line
+	1850 6350 1500 6350
+Wire Wire Line
+	900  6350 900  6850
+Wire Wire Line
+	900  6850 3150 6850
+Connection ~ 3150 6850
+Wire Wire Line
+	3050 3300 900  3300
+Wire Wire Line
+	3050 1700 3050 3300
+Wire Wire Line
+	1550 4000 1550 2050
+Wire Wire Line
+	900  2050 1550 2050
+Connection ~ 1550 2050
+Wire Wire Line
+	1550 2050 1800 2050
 $EndSCHEMATC

Commit message: Add GND and PWR net
Parts:
- removed RELAY1: 6pinRelay, Relay_THT, symbol SchemaBoard_Library:6pinRelay
- added GND2: GND, symbol SchemaBoard_Library:GND
- renumbered GND to GND1, LDR1 to LDR2
Connections:
- net +3V3: no longer GND1.1 (GND)
- net at U1-8.7: now also SW1.2 (D)
- net GND: now reaches U1-8.8
- net GND: now also C1.1, GND1.1 (GND), LDR2.2, GND2.1 (GND)
Changed lines of the file:
@@
 EESchema Schematic File Version 4
+LIBS:circuit3-cache
 EELAYER 29 0
 EELAYER END
@@
 $EndComp
 $Comp
-L SchemaBoard_Library:R_PHOTO LDR1
+L SchemaBoard_Library:R_PHOTO LDR2
 U 1 1 5D3CE114
 P 4300 2050
-F 0 "LDR1" V 3975 2050 50  0000 C CNN
+F 0 "LDR2" V 3975 2050 50  0000 C CNN
 F 1 "R_PHOTO" V 4066 2050 50  0000 C CNN
 F 2 "" V 4350 1800 50  0001 L CNN
@@
 $EndComp
 $Comp
-L SchemaBoard_Library:6pinRelay RELAY1
-U 1 1 5D3E2F18
-P 4700 3750
-F 0 "RELAY1" V 4033 3750 50  0000 C CNN
-F 1 "6pinRelay" V 4124 3750 50  0000 C CNN
-F 2 "Relay_THT" H 5200 3650 50  0001 L CNN
-F 3 "https://standexelectronics.com/wp-content/uploads/datasheet_reed_relay_DIP.pdf" H 4600 3750 50  0001 C CNN
-	1    4700 3750
-	0    1    1    0
-$EndComp
-$Comp
 L SchemaBoard_Library:8pinChip U1-8
 U 1 1 5D3CCD89
@@
 $EndComp
 $Comp
-L SchemaBoard_Library:GND GND
+L SchemaBoard_Library:GND GND1
 U 1 1 5D3D0965
-P 1550 4000
-F 0 "GND" H 1550 3750 50  0001 C CNN
-F 1 "GND" H 1555 3827 50  0000 C CNN
-F 2 "" H 1550 4000 50  0001 C CNN
-F 3 "" H 1550 4000 50  0001 C CNN
-	1    1550 4000
+P 2650 4000
+F 0 "GND1" H 2650 3750 50  0001 C CNN
+F 1 "GND" H 2655 3827 50  0000 C CNN
+F 2 "" H 2650 4000 50  0001 C CNN
+F 3 "" H 2650 4000 50  0001 C CNN
+	1    2650 4000
 	1    0    0    -1
 $EndComp
@@
 $EndComp
 Wire Wire Line
-	2100 2050 4150 2050
+	2100 2050 2650 2050
 Wire Wire Line
 	900  2050 900  3300
@@
 Wire Wire Line
 	7350 3750 7350 5300
-Wire Wire Line
-	5000 3450 6100 3450
-Wire Wire Line
-	6100 3750 5500 3750
-Wire Wire Line
-	5500 3750 5500 4150
-Wire Wire Line
-	5500 4150 5000 4150
-Wire Wire Line
-	4400 4150 4200 4150
-Wire Wire Line
-	4200 4150 4200 5650
 Wire Wire Line
 	4200 5650 3950 5650
@@
 	3050 1700 3050 3300
 Wire Wire Line
-	1550 4000 1550 2050
-Wire Wire Line
-	900  2050 1550 2050
-Connection ~ 1550 2050
-Wire Wire Line
-	1550 2050 1800 2050
+	2650 4000 2650 2050
+$Comp
+L SchemaBoard_Library:GND GND2
+U 1 1 5D454AC6
+P 4900 4700
+F 0 "GND2" H 4900 4450 50  0001 C CNN
+F 1 "GND" H 4988 4663 50  0000 L CNN
+F 2 "" H 4900 4700 50  0001 C CNN
+F 3 "" H 4900 4700 50  0001 C CNN
+	1    4900 4700
+	1    0    0    -1
+$EndComp
+Wire Wire Line
+	4200 3750 6100 3750
+Wire Wire Line
+	4200 3750 4200 5650
+Wire Wire Line
+	4900 3900 4900 4700
+Wire Wire Line
+	4900 3900 6100 3900
+Connection ~ 2650 2050
+Wire Wire Line
+	2650 2050 4150 2050
+Wire Wire Line
+	900  2050 1800 2050
 $EndSCHEMATC

Commit message: In progress: tutorial
Parts:
- renumbered D1 to D3
Other:
- moved on the sheet: SW1A
Changed lines of the file:
@@
 $EndComp
 $Comp
-L SchemaBoard_Library:Diode D1
+L SchemaBoard_Library:Diode D3
 U 1 1 5D3E50B4
 P 2400 5650
-F 0 "D1" H 2400 5866 50  0000 C CNN
+F 0 "D3" H 2400 5866 50  0000 C CNN
 F 1 "Diode" H 2400 5775 50  0000 C CNN
 F 2 "" H 2400 5650 50  0001 C CNN
 F 3 "~" H 2400 5650 50  0001 C CNN
 	1    2400 5650
-	1    0    0    -1
-$EndComp
-$Comp
-L SchemaBoard_Library:SwitchPush SW1
-U 1 1 5D3E6FAF
-P 3750 5650
-F 0 "SW1" H 3750 5935 50  0000 C CNN
-F 1 "SwitchPush" H 3750 5844 50  0000 C CNN
-F 2 "" H 3750 5850 50  0001 C CNN
-F 3 "~" H 3750 5850 50  0001 C CNN
-	1    3750 5650
 	1    0    0    -1
 $EndComp
@@
 	7350 3750 7350 5300
 Wire Wire Line
-	4200 5650 3950 5650
-Wire Wire Line
 	5650 6150 7350 6150
 Connection ~ 7350 6150
@@
 Wire Wire Line
 	3150 6850 3150 5650
-Wire Wire Line
-	3150 5650 3550 5650
 Wire Wire Line
 	7100 3900 7850 3900
@@
 L SchemaBoard_Library:GND GND2
 U 1 1 5D454AC6
-P 4900 4700
-F 0 "GND2" H 4900 4450 50  0001 C CNN
-F 1 "GND" H 4988 4663 50  0000 L CNN
-F 2 "" H 4900 4700 50  0001 C CNN
-F 3 "" H 4900 4700 50  0001 C CNN
-	1    4900 4700
+P 5100 4500
+F 0 "GND2" H 5100 4250 50  0001 C CNN
+F 1 "GND" H 5188 4463 50  0000 L CNN
+F 2 "" H 5100 4500 50  0001 C CNN
+F 3 "" H 5100 4500 50  0001 C CNN
+	1    5100 4500
 	1    0    0    -1
 $EndComp
-Wire Wire Line
-	4200 3750 6100 3750
-Wire Wire Line
-	4200 3750 4200 5650
-Wire Wire Line
-	4900 3900 4900 4700
-Wire Wire Line
-	4900 3900 6100 3900
 Connection ~ 2650 2050
 Wire Wire Line
@@
 Wire Wire Line
 	900  2050 1800 2050
+Wire Wire Line
+	4700 5650 4700 3750
+Wire Wire Line
+	4700 3750 6100 3750
+$Comp
+L SchemaBoard_Library:SwitchPush SW1
+U 1 1 5D3E6FAF
+P 4000 5650
+F 0 "SW1" H 4000 5935 50  0000 C CNN
+F 1 "SwitchPush" H 4000 5844 50  0000 C CNN
+F 2 "" H 4000 5850 50  0001 C CNN
+F 3 "~" H 4000 5850 50  0001 C CNN
+	1    4000 5650
+	1    0    0    -1
+$EndComp
+Wire Wire Line
+	3150 5650 3800 5650
+Wire Wire Line
+	4200 5650 4700 5650
+Wire Wire Line
+	6100 3900 5100 3900
+Wire Wire Line
+	5100 3900 5100 4500
 $EndSCHEMATC

Commit message: In progress: travel net lists
Parts:
- removed BT1: Battery_Cell, symbol SchemaBoard_Library:Battery_Cell
- removed C1: C, symbol SchemaBoard_Library:C
- removed CP1: CP, symbol SchemaBoard_Library:CP
- removed D3: Diode, symbol SchemaBoard_Library:Diode
- removed GND1, GND2: GND, symbol SchemaBoard_Library:GND
- removed L1: Inductor, symbol SchemaBoard_Library:Inductor
- removed LDR2: R_PHOTO, symbol SchemaBoard_Library:R_PHOTO
- removed OPAMP1: OpAmp, symbol SchemaBoard_Library:OpAmp
- removed PWR1: +3.3V, symbol SchemaBoard_Library:+3.3V
- removed Q1: Transistor, symbol SchemaBoard_Library:Transistor
- removed R1: Resistor, symbol SchemaBoard_Library:Resistor
- removed SP1: Speaker, symbol SchemaBoard_Library:Speaker
- removed SW1: SwitchPush, symbol SchemaBoard_Library:SwitchPush
- removed U1-8: 8pinChip, symbol SchemaBoard_Library:8pinChip
- added U1-8: LM555, symbol SchemaBoard_Library:LM555
Connections:
- net at LED1.2 (A): now also U1-8.7 (DIS)
- net at LED1.1 (K): now also U1-8.2 (TR)
