File: software/SchemaBoard_kiCadParser/test timer/555 timer_flip-flop(10).sch (KiCad schematic (older format))
At the start: 12 parts, among them SW3 SwitchPush, SW4 SwitchPush, U1 LM555

Commit message: Add values in the schematic
Parts:
- C2: value C -> 0.01μF; symbol SchemaBoard_Library:C -> schemaboard:C
- GND100: renamed from GND?; symbol SchemaBoard_Library:GND -> schemaboard:GND
- LED10, LED9: symbol SchemaBoard_Library:LED -> schemaboard:LED
- PWR200: renamed from PWR?; value +3.3V -> +9V; symbol SchemaBoard_Library:+3.3V -> schemaboard:+9V
- R5, R6: value Resistor -> 10K; symbol SchemaBoard_Library:Resistor -> schemaboard:Resistor
- R7, R8: value Resistor -> 220; symbol SchemaBoard_Library:Resistor -> schemaboard:Resistor
- SW3: symbol SchemaBoard_Library:SwitchPush -> schemaboard:SwitchPush
- SW4: value SwitchPush -> button; symbol SchemaBoard_Library:SwitchPush -> schemaboard:SwitchPush
- U1-8: renamed from U1; value LM555 -> LM555 Timer; symbol SchemaBoard_Library:LM555 -> schemaboard:LM555
Connections:
- net +3V3 renamed +9V
Other:
- moved on the sheet: C2, LED10, LED9, R5, R6, R7, R8, SW3A, SW4A, U1-8
