File: software/SchemaBoard_kiCadParser/timer_RC.sch (KiCad schematic (older format))
At the start: 13 parts, among them SW11 SwitchPush, U1-8 LM555

Commit message: Add explanation for tutorial
Parts:
- removed GND20: GND-SchemaBoard_Library-555-timer_RC-rescue, symbol timer_RC-rescue:GND-SchemaBoard_Library-555-timer_RC-rescue
- removed PWR30: +3.3V-SchemaBoard_Library-555-timer_RC-rescue, symbol timer_RC-rescue:+3.3V-SchemaBoard_Library-555-timer_RC-rescue
- C10: value C -> 0.033μF; symbol timer_RC-rescue:C-SchemaBoard_Library-555-timer_RC-rescue -> schemaboard:C
- C9: value C -> 0.01μF; symbol timer_RC-rescue:C-SchemaBoard_Library-555-timer_RC-rescue -> schemaboard:C
- CP6: value CP -> 10μF; symbol timer_RC-rescue:CP-SchemaBoard_Library-555-timer_RC-rescue -> schemaboard:CP
- CP7: value CP -> 47μF; symbol timer_RC-rescue:CP-SchemaBoard_Library-555-timer_RC-rescue -> schemaboard:CP
- R2: value Resistor -> 1K minimum; symbol timer_RC-rescue:Resistor-SchemaBoard_Library-555-timer_RC-rescue -> schemaboard:Resistor
- R3: value Resistor -> 47; symbol timer_RC-rescue:Resistor-SchemaBoard_Library-555-timer_RC-rescue -> schemaboard:Resistor
- R4, R5: value Resistor -> 4.7K; symbol timer_RC-rescue:Resistor-SchemaBoard_Library-555-timer_RC-rescue -> schemaboard:Resistor
- SP8: symbol timer_RC-rescue:Speaker-SchemaBoard_Library-555-timer_RC-rescue -> schemaboard:Speaker
- SW11: symbol timer_RC-rescue:SwitchPush-SchemaBoard_Library-555-timer_RC-rescue -> schemaboard:SwitchPush
- U1: renamed from U1-8; value LM555 -> LM555 Timer; symbol timer_RC-rescue:LM555-SchemaBoard_Library-555-timer_RC-rescue -> schemaboard:LM555
Connections:
- net GND: now also R2.2; no longer R2.1
- net at CP7.2, U1.4 (R): now also R2.1; no longer R2.2
- net +3V3 renamed +9V
Other:
- moved on the sheet: C10, C9, CP6, CP7, R2, R3, R4, R5, SP8, SW11A, U1

Commit message: Add values in the schematic
Parts:
- added GND0100: GND, symbol schemaboard:GND
- added PWR0200: +9V, symbol schemaboard:+9V
Connections:
- net +9V: now also PWR0200.1 (+9V)
- net GND: now also GND0100.1 (GND)
Changed lines of the file:
@@
 	5300 2800 6850 2800
 $Comp
-L schemaboard:+9V #PWR0200
+L schemaboard:+9V PWR0200
 U 1 1 5D59C142
 P 3750 2050
-F 0 "#PWR0200" H 3750 1900 50  0001 C CNN
+F 0 "PWR0200" H 3750 1900 50  0001 C CNN
 F 1 "+9V" H 3838 2087 50  0000 L CNN
 F 2 "" H 3750 2050 50  0001 C CNN
@@
 $EndComp
 $Comp
-L schemaboard:GND #GND0100
+L schemaboard:GND GND0100
 U 1 1 5D59CDA7
 P 1950 2600
-F 0 "#GND0100" H 1950 2350 50  0001 C CNN
+F 0 "GND0100" H 1950 2350 50  0001 C CNN
 F 1 "GND" H 2038 2563 50  0000 L CNN
 F 2 "" H 1950 2600 50  0001 C CNN

Commit message: Bugfix tutorial selected icons
Parts:
- SW11: value SwitchPush -> button
Other:
- moved on the sheet: C10, C9, CP6, CP7, R2, R3, R4, R5, SP8, SW11A, U1
