File: software/SchemaBoard_kiCadParser/FlipFlop.sch (KiCad schematic (older format))
At the start: 10 parts, among them SW3 button, SW4 button, U1-8 LM555 Timer

Commit message: change tutorial to guide mode
Parts:
- added GND100: GND, symbol schemaboard:GND
- added PWR200: +9V, symbol schemaboard:+9V
- U1-8: symbol schemaboard:LM555 -> FlipFlop-rescue:LM555-schemaboard
Connections:
- net +9V: now also U1-8.8 (VCC), PWR200.1 (+9V); no longer U1-8.4 (R)
- net GND: now also U1-8.1 (GND), U1-8.6 (THR), GND100.1 (GND); no longer U1-8.2 (TR), U1-8.5 (CV)
- net at C2.2: now also U1-8.5 (CV); no longer U1-8.1 (GND)
- net at U1-8.3 (Q): now also LED10.1 (K), LED9.2 (A)
- net at R6.1, SW4.1 (C): now also U1-8.2 (TR); no longer U1-8.6 (THR)
- net at R5.1, SW3.2 (D): now also U1-8.4 (R); no longer U1-8.8 (VCC)
- now unconnected: U1-8.7 (DIS)
Changed lines of the file:
@@
 EESchema Schematic File Version 4
-LIBS:timer_flip-flop-cache
+LIBS:FlipFlop-cache
 EELAYER 29 0
 EELAYER END
@@
 $EndDescr
 $Comp
-L schemaboard:+9V #PWR0200
+L schemaboard:+9V PWR200
 U 1 1 5D4D6C05
 P 1500 2000
-F 0 "#PWR0200" H 1500 1850 50  0001 C CNN
+F 0 "PWR200" H 1500 1850 50  0001 C CNN
 F 1 "+9V" H 1588 2037 50  0000 L CNN
 F 2 "" H 1500 2000 50  0001 C CNN
@@
 $EndComp
 $Comp
-L schemaboard:GND #GND0100
+L schemaboard:GND GND100
 U 1 1 5D4DA759
 P 7300 1950
-F 0 "#GND0100" H 7300 1700 50  0001 C CNN
+F 0 "GND100" H 7300 1700 50  0001 C CNN
 F 1 "GND" H 7388 1913 50  0000 L CNN
 F 2 "" H 7300 1950 50  0001 C CNN
@@
 	4300 5300 4300 5900
 $Comp
-L schemaboard:LM555 U1-8
+L FlipFlop-rescue:LM555-schemaboard U1-8
 U 1 1 5D4D75EC
 P 5300 4250
