File: software/SchemaBoard_kiCadParser/timer_flip-flop.sch (KiCad schematic (older format))
At the start: 12 parts, among them SW3 SwitchPush, SW4 button, U1-8 LM555 Timer

Commit message: Bugfix tutorial selected icons
Parts:
- removed GND0100: GND, symbol schemaboard:GND
- removed PWR0200: +9V, symbol schemaboard:+9V
- SW3: value SwitchPush -> button
Other:
- moved on the sheet: C2, LED10, LED9, R5, R6, R7, R8, SW3A, SW4A, U1-8

Commit message: change tutorial to guide mode
Parts:
- removed LED10: LED, symbol schemaboard:LED
- added LED10: LED, symbol schemaboard:LED2
Connections:
- net +9V: now also U1-8.8 (VCC); no longer U1-8.4 (R)
- net GND: now also U1-8.1 (GND), U1-8.6 (THR); no longer U1-8.2 (TR), U1-8.5 (CV)
- net at C2.2: now also U1-8.5 (CV); no longer U1-8.1 (GND)
- net at U1-8.3 (Q): now also LED9.2 (A), LED10.1 (K)
- net at R6.1, SW4.1 (C): now also U1-8.2 (TR); no longer U1-8.6 (THR)
- net at U1-8.7 (DIS): no longer LED9.2 (A)
- net at R5.1, SW3.2 (D): now also U1-8.4 (R); no longer U1-8.8 (VCC)
- net at R7.1: now also LED10.2 (A)
Other:
- moved on the sheet: U1-8
Changed lines of the file:
@@
-$EndComp
-$Comp
-L schemaboard:LED LED10
-U 1 1 5D4E318A
-P 3250 4300
-F 0 "LED10" H 3243 4045 50  0000 C CNN
-F 1 "LED" H 3243 4136 50  0000 C CNN
-F 2 "" H 3250 4300 50  0001 C CNN
-F 3 "~" H 3250 4300 50  0001 C CNN
-	1    3250 4300
-	-1   0    0    1
 $EndComp
 $Comp
@@
 L schemaboard:LM555 U1-8
 U 1 1 5D4D75EC
-P 5300 4250
-F 0 "U1-8" H 5300 3783 50  0000 C CNN
-F 1 "LM555 Timer" H 5300 3874 50  0000 C CNN
-F 2 "" H 5300 4250 50  0001 C CNN
-F 3 "http://www.ti.com/lit/ds/symlink/lm555.pdf" H 5300 4250 50  0001 C CNN
-	1    5300 4250
-	-1   0    0    1
+P 5300 4200
+F 0 "U1-8" H 5300 3733 50  0000 C CNN
+F 1 "LM555 Timer" H 5300 3824 50  0000 C CNN
+F 2 "" H 5300 4200 50  0001 C CNN
+F 3 "http://www.ti.com/lit/ds/symlink/lm555.pdf" H 5300 4200 50  0001 C CNN
+	1    5300 4200
+	1    0    0    -1
 $EndComp
 Wire Wire Line
@@
 	7300 1950 7300 2650
 Connection ~ 7300 2650
+$Comp
+L schemaboard:LED2 LED10
+U 1 1 5D7B538A
+P 3250 4300
+F 0 "LED10" H 3257 4555 50  0000 C CNN
+F 1 "LED" H 3257 4464 50  0000 C CNN
+F 2 "" H 3250 4300 50  0001 C CNN
+F 3 "~" H 3250 4300 50  0001 C CNN
+	1    3250 4300
+	1    0    0    -1
+$EndComp
 $EndSCHEMATC
